File: Tesla Coil.sch (EAGLE design)
At the start: 9 parts, among them IC1 NE555

Commit message: Driver toegevoegd
Parts:
- added B1: DBDB105G, rectifier:DBDB105G
- added JP4, JP5: (no value), pinhead:PINHD-1X2
- added TR1, TR2, TR3, TR4: 1:33, inductor-neosid:U15-TRANSFORMER
Connections:
- removed net GNDA: C1.2, C2.2, C3.1, IC1.GND, JP1.2, JP2.1
- new net GND: B1.-, C1.2, C2.2, C3.1, IC1.GND, JP1.2, JP2.1
- new net N$10: JP5.1, TR3.1
- new net N$11: JP4.1, TR1.1
- new net N$12: TR3.4, TR4.2
- new net N$13: TR3.3, TR4.1
- new net N$14: B1.AC1, TR2.4
- new net N$15: B1.AC2, TR2.3
- new net N$6: TR1.4, TR2.2
- new net N$7: TR1.3, TR2.1
- new net N$8: JP4.2, TR1.2
- new net N$9: JP5.2, TR3.2

Commit message: Driver
Parts:
- added C10, C11, C6, C7, C8, C9: 100nF, eagle-ltspice:CC0603
- added C4, C5: (no value), eagle-ltspice:CC0603
- added IC2: LM311D, linear:LM311D
- added IC3: LM555D, linear:LM555D
- added IC4: 74HC14D, 74xx-eu:74HC14D
- added LED1: (no value), led:LEDCHIP-LED0603
- added Q1: IRLML6346TRPBF, transistor-power:FDN360P
- added R10, R11, R12, R4, R5, R6, R7, R8, R9: (no value), eagle-ltspice:RR0603
- added R3: (no value), pot:TRIM_EU-3223G
Connections:
- new net 555TRIG: IC2.OUT, R7.2
- new net N$16: IC2.ON, IC2.ON/STR
- new net N$17: B1.+, C4.2, IC2.-IN, R5.1
- new net N$18: C5.2, IC2.+IN, R3.S
- new net N$19: IC3.TR
- new net N$20: R3.E, R6.2
- new net N$21: C7.2, IC3.CV
- new net N$22: C9.2, IC3.DIS, IC3.THR, R8.2
- new net N$23: IC3.Q, Q1.G, R9.1
- new net N$24: LED1.A, R9.2
- new net N$25: R10.2, TR4.4
- new net N$27: C8.1, IC4D.I
- new net N$29: C8.2, R10.1
- new net N$30: IC4D.O, IC4E.I
- new net OCDTRIG: Q1.S
- net GND: now also C10.1, C11.1, C4.1, C5.1, C6.1, C7.1, C9.1, IC2.GND, IC2.V-, IC3.GND, IC4P.GND, LED1.C, Q1.D, R3.A, R5.2, TR4.3
- net N$14: now also R4.2
- net N$15: now also R4.1
- net VCC: now also C10.2, C11.2, C6.2, IC2.V+, IC3.R, IC3.V+, IC4P.VCC, R6.1, R7.1, R8.1
Other:
- moved on the sheet: B1, JP4, JP5, TR1, TR2, TR3, TR4

Commit message: H-Brug V1
Parts:
- added B2: DBDB105G, rectifier:DBDB105G
- added C12, C13: (no value), resistor:CPOL-EUTAP5-45
- added C14: (no value), resistor:C-EUC0603
- added D10, D7, D8, D9: 1N5817-B, diode:1N5817-B
- added JP10, JP6, JP7, JP8, JP9: (no value), pinhead:PINHD-1X2
- added L1: (no value), resistor:L-USL3216C
- added Q2, Q3, Q4, Q5: BUZ60, transistor-fet:BUZ60
- added R13, R14, R15, R16: (no value), resistor:R-EU_R0805
Connections:
- new net GDT1+: D7.C, JP7.2, R13.1
- new net GDT1-: C14.2, JP7.1, Q2.S, Q3.D
- new net GDT2-: D8.C, JP8.2, R14.1
- new net GDT3+: JP9.2, L1.2, Q4.D, Q5.S
- new net GDT3-: D9.C, JP9.1, R15.1
- new net GDT4+: D10.C, JP10.1, R16.1
- new net N$31: B2.AC1, JP6.2
- new net N$32: B2.AC2, JP6.1
- new net N$33: B2.+, C12.+, C13.+, Q2.D, Q4.S
- new net N$35: D9.A, Q4.G, R15.2
- new net N$37: C14.1, L1.1
- new net N$38: Q2.G, R13.2
- new net N$40: D7.A
- new net N$41: D8.A, Q3.G, R14.2
- new net N$42: D10.A, Q5.G, R16.2
- net GND: now also B2.-, C12.-, C13.-, JP10.2, JP8.1, Q3.S, Q5.D
