File: Tesla Coil.sch (EAGLE design)
At the start: 39 parts, among them IC1 NE555, IC2 LM311D, IC3 LM555D, IC4 74HC14D, Q1 IRLML6346TRPBF

Commit message: Driver afgemaakt + ground fix
Parts:
- added C12, C13: 100nF, eagle-ltspice:CC0603
- added D1, D4: 1N4446, diode:1N4446
- added D2, D3: BZX84CSMD, diode:BZX84CSMD
- added IC5: 74HC109N, 74xx-eu:74HC109N
- added JP6: (no value), pinhead:PINHD-1X2
- C11: value 100nF -> 1nF
- C4, C5: value (none) -> 100nF
- C6, C8: value 100nF -> (none)
- IC2: value LM311D -> 74HC14D; device linear:LM311D -> 74xx-eu:74HC14D
- IC3: value LM555D -> LM311D; device linear:LM555D -> linear:LM311D
- IC4: value 74HC14D -> LM555D; device 74xx-eu:74HC14D -> linear:LM555D
- R3: device pot:TRIM_EU-3223G -> eagle-ltspice:RR0603
- R6: device eagle-ltspice:RR0603 -> pot:TRIM_EU-3223G
Connections:
- removed net N$10 (its old number): JP5.1, TR3.1
- removed net N$9 (its old number): JP5.2, TR3.2
- new net +15V: C9.2, IC3.V+, IC4.V+, R11.1, R7.1, R9.1
- new net +5V: C4.2, C5.2, IC2P.VCC, IC5A.J, IC5A.K, IC5P.VCC
- new net CLK: IC2E.O
- new net GDTSIG: IC5A.!Q
- new net N$11: JP5.1, TR2.1
- new net N$26: D1.C, D2.C
- new net N$28: D3.C, D4.C
- new net N$31: JP6.2, R8.2
- new net N$32: IC2C.I, IC2F.I, R8.1
- new net N$33: IC2F.O, R10.2
- new net N$34: C11.2, IC2B.I, R10.1
- new net N$35: IC2C.O, IC5A.CLR
- new net N$36: IC5A.PRE
- new net N$37: IC5A.CLK
- new net N$8: JP5.2, TR2.2
- new net PRE: IC2B.O
- net 555TRIG: now also IC3.OUT, R9.2; no longer IC2.OUT, R7.2
- net GND: now also C1.1, C12.1, C13.1, C3.2, C8.1, D2.A, D4.A, IC2A.I, IC2P.GND, IC3.V-, IC4.GND, IC5B.CLK, IC5B.CLR, IC5B.J, IC5B.K, IC5B.PRE, IC5P.GND, JP1.1, JP3.2, JP6.1, R4.2, R6.A, TR3.3; no longer C1.2, C3.1, C7.1, IC2.GND, IC2.V-, IC4P.GND, JP1.2, JP2.1, R3.A, R5.2, TR4.3
- net N$12: now also TR1.4, TR3.2; no longer TR3.4, TR4.2
- net N$13: now also TR1.3, TR3.1; no longer TR3.3, TR4.1
- net N$14: now also R3.2, TR4.4; no longer R4.2, TR2.4
- net N$15: now also R3.1, TR4.3; no longer R4.1, TR2.3
- net N$16: now also IC3.ON, IC3.ON/STR; no longer IC2.ON, IC2.ON/STR
- net N$17: now also C6.2, IC3.-IN, R4.1; no longer C4.2, IC2.-IN, R5.1
- net N$18: now also C8.2, IC3.+IN, R6.S; no longer C5.2, IC2.+IN, R3.S
- net N$19: now also IC4.TR; no longer IC3.TR
- net N$2: now also C2.1; no longer C1.1
- net N$20: now also R6.E, R7.2; no longer R3.E, R6.2
- net N$21: now also C12.2, IC4.CV; no longer C7.2, IC3.CV
- net N$22: now also C13.2, IC4.DIS, IC4.THR, R11.2; no longer C9.2, IC3.DIS, IC3.THR, R8.2
- net N$23: now also IC4.Q, R12.1; no longer IC3.Q, R9.1
- net N$24: now also R12.2; no longer R9.2
- net N$25: now also D1.A, D3.A, R5.2, TR3.4; no longer R10.2, TR4.4
- net N$27: now also C7.1, IC2D.I; no longer C8.1, IC4D.I
- net N$29: now also C7.2, R5.1; no longer C8.2, R10.1
- net N$3: now also C3.1; no longer C2.1
- net N$30: now also IC2D.O, IC2E.I; no longer IC4D.O, IC4E.I
- net N$4: now also C1.2, JP1.2; no longer C3.2, JP3.2
- net N$5: now also JP3.1; no longer JP1.1
- net N$6: now also TR2.4, TR4.2; no longer TR1.4, TR2.2
- net N$7: now also TR2.3, TR4.1; no longer TR1.3, TR2.1
- net VCC: now also IC4.R, JP2.1; no longer C11.2, C6.2, IC2.V+, IC3.R, IC3.V+, IC4P.VCC, JP3.1, R6.1, R7.1, R8.1
Other:
- moved on the sheet: C1, C11, C2, C3, C4, C5, C6, C7, C8, C9, JP1, JP2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
